Commit message: Added wheels

File: urdf/my_robot.xacro (robot description, xacro)
@@ -55,3 +55,65 @@
     </visual>
   </link>
+  <link name='left_wheel'>
+    <inertial>
+      <mass value="5.0"/>
+      <origin xyz="0 0 0" rpy="0 1.5707 1.5707"/>
+      <inertia
+          ixx="0.1" ixy="0" ixz="0"
+          iyy="0.1" iyz="0"
+          izz="0.1"
+      />
+    </inertial>
+    <collision name='collision'>
+      <origin xyz="0 0 0" rpy="0 1.5707 1.5707"/>
+      <geometry>
+        <box size=".4 .2 .1"/>
+      </geometry>
+    </collision>
+    <visual name='wheel_visual'>
+      <origin xyz="0 0 0" rpy="0 1.5707 1.5707"/>
+      <geometry>
+        <cylinder length="0.05" radius="0.1" />
+      </geometry>
+    </visual>
+  </link>
+  <link name='right_wheel'>
+    <inertial>
+      <mass value="5.0"/>
+      <origin xyz="0 0 0" rpy="0 1.5707 1.5707"/>
+      <inertia
+          ixx="0.1" ixy="0" ixz="0"
+          iyy="0.1" iyz="0"
+          izz="0.1"
+      />
+    </inertial>
+    <collision name='collision'>
+      <origin xyz="0 0 0" rpy="0 1.5707 1.5707"/>
+      <geometry>
+        <box size=".4 .2 .1"/>
+      </geometry>
+    </collision>
+    <visual name='wheel_visual'>
+      <origin xyz="0 0 0" rpy="0 1.5707 1.5707"/>
+      <geometry>
+        <cylinder length="0.05" radius="0.1" />
+      </geometry>
+    </visual>
+  </link>
+  <joint type="continuous" name="left_wheel_hinge">
+    <origin xyz="0 0.15 0" rpy="0 0 0"/>
+    <child link="left_wheel"/>
+    <parent link="chassis"/>
+    <axis xyz="0 1 0" rpy="0 0 0"/>
+    <limit effort="10000" velocity="1000"/>
+    <dynamics damping="1.0" friction="1.0"/>
+  </joint>
+  <joint type="continuous" name="right_wheel_hinge">
+    <origin xyz="0 -0.15 0" rpy="0 0 0"/>
+    <child link="right_wheel"/>
+    <parent link="chassis"/>
+    <axis xyz="0 1 0" rpy="0 0 0"/>
+    <limit effort="10000" velocity="1000"/>
+    <dynamics damping="1.0" friction="1.0"/>
+  </joint>
 </robot>

Commit message: Added camera and lidar sensor links/joints

File: urdf/my_robot.xacro (robot description, xacro)
@@ -29,4 +29,5 @@
         <box size=".4 .2 .1"/>
       </geometry>
+      <material name="white"/>
     </visual>
     <collision name='back_caster_collision'>
@@ -41,4 +42,5 @@
         <sphere radius="0.05"/>
       </geometry>
+      <material name="white"/>
     </visual>
     <collision name='front_caster_collision'>
@@ -53,4 +55,5 @@
         <sphere radius="0.05"/>
       </geometry>
+      <material name="white"/>
     </visual>
   </link>
@@ -65,5 +68,5 @@
       />
     </inertial>
-    <collision name='collision'>
+    <collision>
       <origin xyz="0 0 0" rpy="0 1.5707 1.5707"/>
       <geometry>
@@ -71,9 +74,10 @@
       </geometry>
     </collision>
-    <visual name='wheel_visual'>
+    <visual>
       <origin xyz="0 0 0" rpy="0 1.5707 1.5707"/>
       <geometry>
         <cylinder length="0.05" radius="0.1" />
       </geometry>
+      <material name="green"/>
     </visual>
   </link>
@@ -88,5 +92,5 @@
       />
     </inertial>
-    <collision name='collision'>
+    <collision>
       <origin xyz="0 0 0" rpy="0 1.5707 1.5707"/>
       <geometry>
@@ -94,9 +98,10 @@
       </geometry>
     </collision>
-    <visual name='wheel_visual'>
+    <visual>
       <origin xyz="0 0 0" rpy="0 1.5707 1.5707"/>
       <geometry>
         <cylinder length="0.05" radius="0.1" />
       </geometry>
+      <material name="green"/>
     </visual>
   </link>
@@ -117,3 +122,63 @@
     <dynamics damping="1.0" friction="1.0"/>
   </joint>
+  <link name='camera'>
+    <inertial>
+      <mass value=".1"/>
+      <origin xyz=".05 .05 .05" rpy="0 0 0"/>
+      <inertia
+          ixx="1e-6" ixy="0" ixz="0"
+          iyy="1e-6" iyz="0"
+          izz="1e-6"
+      />
+    </inertial>
+    <collision>
+      <origin xyz="0 0 0" rpy="0 0 0"/>
+      <geometry>
+        <box size=".05 .05 .05" />
+      </geometry>
+    </collision>
+    <visual>
+      <origin xyz="0 0 0" rpy="0 0 0"/>
+      <geometry>
+        <box size=".05 .05 .05" />
+      </geometry>
+      <material name="red"/>
+    </visual>
+  </link>
+  <joint name="camera_joint" type="fixed">
+    <origin xyz=".2 0 0" rpy="0 0 0" />
+    <parent link="chassis"/>
+    <child link="camera" />
+    <axis xyz="0 1 0" rpy="0 0 0"/>
+  </joint>
+  <link name='hokuyo'>
+    <inertial>
+      <mass value="1e-5"/>
+      <origin xyz="0 0 0" rpy="0 0 0"/>
+      <inertia
+          ixx="1e-6" ixy="0" ixz="0"
+          iyy="1e-6" iyz="0"
+          izz="1e-6"
+      />
+    </inertial>
+    <collision>
+      <origin xyz="0 0 0" rpy="0 0 0"/>
+      <geometry>
+        <box size=".1 .1 .1" />
+      </geometry>
+    </collision>
+    <visual>
+      <origin xyz="0 0 0" rpy="0 0 0"/>
+      <geometry>
+        <mesh filename="package://my_robot/meshes/hokuyo.dae"/>
+      </geometry>
+      <material name="grey"/>
+    </visual>
+  </link>
+  <joint name="hokuyo_joint" type="fixed">
+    <origin xyz=".15 0 .1" rpy="0 0 0" />
+    <parent link="chassis"/>
+    <child link="hokuyo" />
+    <axis xyz="0 1 0" rpy="0 0 0"/>
+  </joint>
 </robot>

Commit message: Added material definitions

File: urdf/my_robot.xacro (robot description, xacro)
@@ -1,4 +1,9 @@
 <?xml version='1.0'?>
 <robot name="my_robot" xmlns:xacro="http://www.ros.org/wiki/xacro">
+  <material name="white"> <color rgba="1 1 1 1"/></material>
+  <material name="grey">  <color rgba=".6 .6 .6 1"/></material>
+  <material name="red">   <color rgba="1 0 0 1"/></material>
+  <material name="green"> <color rgba="0 1 0 1"/></material>
+  <material name="blue">  <color rgba="0 0 1 1"/></material>
   <link name="robot_footprint"></link>
   <joint name="robot_footprint_joint" type="fixed">

Commit message: Removed obsolete axis from fixed joints

File: urdf/my_robot.xacro (robot description, xacro)
@@ -155,5 +155,4 @@
     <parent link="chassis"/>
     <child link="camera" />
-    <axis xyz="0 1 0" rpy="0 0 0"/>
   </joint>
   <link name='hokuyo'>
@@ -185,5 +184,4 @@
     <parent link="chassis"/>
     <child link="hokuyo" />
-    <axis xyz="0 1 0" rpy="0 0 0"/>
   </joint>
 </robot>

Commit message: Color using gazebo element

File: urdf/my_robot.xacro (robot description, xacro)
@@ -185,3 +185,5 @@
     <child link="hokuyo" />
   </joint>
+  <gazebo reference="left_wheel"><material>Gazebo/Green</material></gazebo>
+  <gazebo reference="right_wheel"><material>Gazebo/Green</material></gazebo>
 </robot>

Commit message: Color using gazebo element

File: urdf/my_robot.xacro (robot description, xacro)
@@ -1,9 +1,4 @@
 <?xml version='1.0'?>
 <robot name="my_robot" xmlns:xacro="http://www.ros.org/wiki/xacro">
-  <material name="white"> <color rgba="1 1 1 1"/></material>
-  <material name="grey">  <color rgba=".6 .6 .6 1"/></material>
-  <material name="red">   <color rgba="1 0 0 1"/></material>
-  <material name="green"> <color rgba="0 1 0 1"/></material>
-  <material name="blue">  <color rgba="0 0 1 1"/></material>
   <link name="robot_footprint"></link>
   <joint name="robot_footprint_joint" type="fixed">
@@ -34,5 +29,4 @@
         <box size=".4 .2 .1"/>
       </geometry>
-      <material name="white"/>
     </visual>
     <collision name='back_caster_collision'>
@@ -47,5 +41,4 @@
         <sphere radius="0.05"/>
       </geometry>
-      <material name="white"/>
     </visual>
     <collision name='front_caster_collision'>
@@ -60,5 +53,4 @@
         <sphere radius="0.05"/>
       </geometry>
-      <material name="white"/>
     </visual>
   </link>
@@ -84,5 +76,4 @@
         <cylinder length="0.05" radius="0.1" />
       </geometry>
-      <material name="green"/>
     </visual>
   </link>
@@ -108,5 +99,4 @@
         <cylinder length="0.05" radius="0.1" />
       </geometry>
-      <material name="green"/>
     </visual>
   </link>
@@ -148,5 +138,4 @@
         <box size=".05 .05 .05" />
       </geometry>
-      <material name="red"/>
     </visual>
   </link>
@@ -177,5 +166,4 @@
         <mesh filename="package://my_robot/meshes/hokuyo.dae"/>
       </geometry>
-      <material name="grey"/>
     </visual>
   </link>
@@ -187,3 +175,4 @@
   <gazebo reference="left_wheel"><material>Gazebo/Green</material></gazebo>
   <gazebo reference="right_wheel"><material>Gazebo/Green</material></gazebo>
+  <gazebo reference="camera"><material>Gazebo/Red</material></gazebo>
 </robot>
