Commit message: Fixed robot collision geometry

File: my_robot/urdf/my_robot.xacro (robot description, xacro)
@@ -69,5 +69,5 @@
       <origin xyz="0 0 0" rpy="0 1.5707 1.5707"/>
       <geometry>
-        <box size=".4 .2 .1"/>
+        <cylinder length="0.05" radius="0.1" />
       </geometry>
     </collision>
@@ -92,5 +92,5 @@
       <origin xyz="0 0 0" rpy="0 1.5707 1.5707"/>
       <geometry>
-        <box size=".4 .2 .1"/>
+        <cylinder length="0.05" radius="0.1" />
       </geometry>
     </collision>

Commit message: Made changes to robot geometry

File: my_robot/urdf/my_robot.xacro (robot description, xacro)
@@ -22,5 +22,5 @@
       <origin xyz="0 0 0" rpy=" 0 0 0"/>
       <geometry>
-        <box size=".4 .2 .1"/>
+        <box size=".5 .2 .3"/>
       </geometry>
     </collision>
@@ -28,9 +28,9 @@
       <origin xyz="0 0 0" rpy=" 0 0 0"/>
       <geometry>
-        <box size=".4 .2 .1"/>
+        <box size=".5 .2 .3"/>
       </geometry>
     </visual>
     <collision name='back_caster_collision'>
-      <origin xyz="-0.15 0 -0.05" rpy=" 0 0 0"/>
+      <origin xyz="-0.2 0 -0.15" rpy=" 0 0 0"/>
       <geometry>
         <sphere radius="0.0499"/>
@@ -38,5 +38,5 @@
     </collision>
     <visual name='back_caster_visual'>
-      <origin xyz="-0.15 0 -0.05" rpy=" 0 0 0"/>
+      <origin xyz="-0.2 0 -0.15" rpy=" 0 0 0"/>
       <geometry>
         <sphere radius="0.05"/>
@@ -44,5 +44,5 @@
     </visual>
     <collision name='front_caster_collision'>
-      <origin xyz="0.15 0 -0.05" rpy=" 0 0 0"/>
+      <origin xyz="0.2 0 -0.15" rpy=" 0 0 0"/>
       <geometry>
         <sphere radius="0.0499"/>
@@ -50,5 +50,5 @@
     </collision>
     <visual name='front_caster_visual'>
-      <origin xyz="0.15 0 -0.05" rpy=" 0 0 0"/>
+      <origin xyz="0.2 0 -0.15" rpy=" 0 0 0"/>
       <geometry>
         <sphere radius="0.05"/>
@@ -69,5 +69,5 @@
       <origin xyz="0 0 0" rpy="0 1.5707 1.5707"/>
       <geometry>
-        <cylinder length="0.05" radius="0.1" />
+        <cylinder length="0.05" radius="0.2" />
       </geometry>
     </collision>
@@ -75,5 +75,5 @@
       <origin xyz="0 0 0" rpy="0 1.5707 1.5707"/>
       <geometry>
-        <cylinder length="0.05" radius="0.1" />
+        <cylinder length="0.05" radius="0.2" />
       </geometry>
     </visual>
@@ -92,5 +92,5 @@
       <origin xyz="0 0 0" rpy="0 1.5707 1.5707"/>
       <geometry>
-        <cylinder length="0.05" radius="0.1" />
+        <cylinder length="0.05" radius="0.2" />
       </geometry>
     </collision>
@@ -98,5 +98,5 @@
       <origin xyz="0 0 0" rpy="0 1.5707 1.5707"/>
       <geometry>
-        <cylinder length="0.05" radius="0.1" />
+        <cylinder length="0.05" radius="0.2" />
       </geometry>
     </visual>
@@ -142,5 +142,5 @@
   </link>
   <joint name="camera_joint" type="fixed">
-    <origin xyz=".2 0 0" rpy="0 0 0" />
+    <origin xyz=".25 0 0" rpy="0 0 0" />
     <parent link="chassis"/>
     <child link="camera" />
@@ -170,10 +170,11 @@
   </link>
   <joint name="hokuyo_joint" type="fixed">
-    <origin xyz=".15 0 .1" rpy="0 0 0" />
+    <origin xyz=".2 0 .15" rpy="0 0 0" />
     <parent link="chassis"/>
     <child link="hokuyo" />
   </joint>
-  <gazebo reference="left_wheel"><material>Gazebo/Green</material></gazebo>
-  <gazebo reference="right_wheel"><material>Gazebo/Green</material></gazebo>
+  <gazebo reference="left_wheel"><material>Gazebo/Blue</material></gazebo>
+  <gazebo reference="right_wheel"><material>Gazebo/Blue</material></gazebo>
+  <gazebo reference="chassis"><material>Gazebo/Green</material></gazebo>
   <gazebo reference="camera"><material>Gazebo/Red</material></gazebo>
 </robot>
